Commit message: Fix URDF link name casing and update USD path; refactor command configurations and reward functions for consistency

File: kanake6_sim_523/kanake6_sim_0808_4.SLDASM/urdf/kanake6_sim_0808_4.SLDASM.urdf (robot description, URDF)
Before this commit: robot kanake6_sim_0808_4.SLDASM, 17 links, 16 joints
Links:
- removed link LInk11
- added link Link11, mass 0.0712511533582805; collision mesh filename=package://kanake6_sim_0808_4.SLDASM/meshes/Link11.STL; visual mesh filename=package://kanake6_sim_0808_4.SLDASM/meshes/Link11.STL
Joints:
- joint j11: child LInk11 -> Link11
- joint j12: parent LInk11 -> Link11
